Commit message: added my own custom world

File: urdf/robot.xacro (robot description, xacro)
@@ -37,5 +37,5 @@
       <origin xyz="-0.15 0 -0.05" rpy=" 0 0 0"/>
       <geometry>
-        <sphere radius="0.045"/>
+        <sphere radius="0.049"/>
       </geometry>
       <surface>
@@ -53,5 +53,5 @@
       <origin xyz="-0.15 0 -0.05" rpy=" 0 0 0"/>
       <geometry>
-        <sphere radius="0.045"/>
+        <sphere radius="0.049"/>
       </geometry>
       <material name="Cyan">
@@ -62,5 +62,5 @@
       <origin xyz="0.15 0 -0.05" rpy=" 0 0 0"/>
       <geometry>
-        <sphere radius="0.045"/>
+        <sphere radius="0.049"/>
       </geometry>
       <surface>
@@ -78,5 +78,5 @@
       <origin xyz="0.15 0 -0.05" rpy=" 0 0 0"/>
       <geometry>
-        <sphere radius="0.045"/>
+        <sphere radius="0.049"/>
       </geometry>
       <material name="Cyan">

Commit message: fixed 3d mapping

File: urdf/robot.xacro (robot description, xacro)
@@ -180,5 +180,22 @@
     <origin xyz="0.2 0 0" rpy="0 0 0"/>
     <child link="camera"/>
-    <parent link="chassis"/>
+    <parent link="robot_footprint"/>
+  </joint>
+  <link name='camera_depth'>
+    <visual name='chassis_visual'>
+      <origin xyz="0 0 0" rpy="0 0 0"/>
+      <geometry>
+        <box size="0.05 0.05 0.05"/>
+      </geometry>
+      <material name="Cyan">
+        <color rgba="0 1.0 1.0 1.0"/>
+      </material>
+    </visual>
+  </link>
+  <!--joint type="continuous" name="left_wheel_hinge"-->
+  <joint type="fixed" name="camera_joint_correction">
+    <origin xyz="0 0 0" rpy="1.57 3.14 1.57"/>
+    <child link="camera_depth"/>
+    <parent link="camera"/>
   </joint>
   <!-- hokuyo -->
